Commit message: [Add] plate & torque response test in mujoco

File: fr3_husky_description/mjcf/dual_fr3.xml.xacro (robot description, xacro)
@@ -21,4 +21,5 @@
     <xacro:include filename="$(find fr3_husky_description)/mjcf/assets/d435i_assets.xml.xacro"/>
     <xacro:include filename="$(find fr3_husky_description)/mjcf/assets/azure_kinect_assets.xml.xacro"/>
+    <xacro:include filename="$(find fr3_husky_description)/mjcf/plate_ee.xml.xacro"/>
     <!-- ============================================================= -->
     <!-- Should an end-effector be mounted at the flange? -->
@@ -50,4 +51,12 @@
                     value="${'0 0 0.523598776;0 0 -0.523598776' if '$(arg mobile)' == 'true' else '0 0 0;0 0 0'}" />
     <xacro:arg name="control_mode" default="effort" />
+    <!-- The reach launch uses hand=false. In that configuration use the
+         effective link7 inertia from Isaac's dual_fr3_plate_ee.usd. -->
+    <xacro:property name="standard_fr3_inertials"
+                    value="${xacro.load_yaml('$(find franka_description)/mjcf/robots/fr3/inertials.yaml')}" />
+    <xacro:property name="isaac_reach_fr3_inertials"
+                    value="${xacro.load_yaml('$(find fr3_husky_description)/config/fr3_isaac_reach_inertials.yaml')}" />
+    <xacro:property name="fr3_arm_inertials"
+                    value="${standard_fr3_inertials if '$(arg hand)' == 'true' else isaac_reach_fr3_inertials}" />
     <xacro:property name="ee2cam_left_tf"
                     value="${xacro.load_yaml('$(find fr3_husky_description)/config/TF_ee2cam_left.yaml')}" />
@@ -67,5 +76,5 @@
             joint_limits="${xacro.load_yaml('$(find franka_description)/mjcf/robots/fr3/joint_limits.yaml')}"
             kinematics="${xacro.load_yaml('$(find franka_description)/mjcf/robots/fr3/kinematics.yaml')}"
-            inertials="${xacro.load_yaml('$(find franka_description)/mjcf/robots/fr3/inertials.yaml')}"
+            inertials="${fr3_arm_inertials}"
             dynamics="${xacro.load_yaml('$(find franka_description)/mjcf/robots/fr3/dynamics.yaml')}"
             accelerometer_config="${xacro.load_yaml('$(find franka_description)/mjcf/robots/fr3/accelerometers.yaml')}"
@@ -97,4 +106,7 @@
             finger_vis_mesh_materials="['off_white','black']">
             <cam_body>
+                <xacro:unless value="$(arg hand)">
+                    <xacro:plate_ee_mjcf prefix="${arm_prefix}_fr3"/>
+                </xacro:unless>
                 <xacro:if value="$(arg with_realsense)">
                     <xacro:realsense_d435i_mjcf prefix="${arm_prefix}" ee2cam_tf="${ee2cam_tf}"
@@ -110,5 +122,6 @@
     <compiler angle="radian" autolimits="true" />
     <!-- ── Option ── -->
-    <option timestep="0.001" integrator="implicitfast" />
+    <!-- Match dual_fr3_lab Reach v2, where gravity is disabled for the robot. -->
+    <option timestep="0.001" integrator="implicitfast" gravity="0 0 0" />
     <!-- ── Visual ── -->
     <visual>
@@ -151,4 +164,5 @@
         <xacro:husky_assets/>
         <xacro:roas_structure_assets/>
+        <xacro:plate_ee_mjcf_assets/>
         <xacro:if value="$(arg with_realsense)">
             <xacro:d435i_assets/>

File: fr3_husky_description/robots/dual_fr3.urdf.xacro (robot description, xacro)
@@ -4,4 +4,5 @@
     <xacro:include filename="$(find fr3_husky_description)/robots/realsense_d435i.urdf.xacro"/>
     <xacro:include filename="$(find fr3_husky_description)/robots/azure_kinect.urdf.xacro"/>
+    <xacro:include filename="$(find fr3_husky_description)/robots/plate_ee.urdf.xacro"/>
     <!-- base xacro includes -->
     <xacro:include filename="$(find fr3_husky_description)/robots/box_base.xacro"/>
@@ -129,3 +130,9 @@
         fix_finger="$(arg fix_finger)"
     />
+    <!-- The reach policy is launched with hand=false; mount the same flat
+         plate geometry used by the Isaac reach asset in that configuration. -->
+    <xacro:unless value="$(arg hand)">
+        <xacro:plate_ee prefix="left_fr3" parent="left_fr3_link8"/>
+        <xacro:plate_ee prefix="right_fr3" parent="right_fr3_link8"/>
+    </xacro:unless>
 </robot>

Commit message: [Fix] test (rollout nominal trajectory for different env&control condition)

File: fr3_husky_description/mjcf/dual_fr3.xml.xacro (robot description, xacro)
@@ -51,4 +51,9 @@
                     value="${'0 0 0.523598776;0 0 -0.523598776' if '$(arg mobile)' == 'true' else '0 0 0;0 0 0'}" />
     <xacro:arg name="control_mode" default="effort" />
+    <!-- Reach dynamics ablation parameters. The launch file generates the
+         dynamics YAML for all seven joints; physics timestep remains 1 ms. -->
+    <xacro:arg name="fr3_armature" default="0.1" />
+    <xacro:arg name="fr3_dynamics_path"
+               default="$(find franka_description)/mjcf/robots/fr3/dynamics.yaml" />
     <!-- The reach launch uses hand=false. In that configuration use the
          effective link7 inertia from Isaac's dual_fr3_plate_ee.usd. -->
@@ -77,5 +82,5 @@
             kinematics="${xacro.load_yaml('$(find franka_description)/mjcf/robots/fr3/kinematics.yaml')}"
             inertials="${fr3_arm_inertials}"
-            dynamics="${xacro.load_yaml('$(find franka_description)/mjcf/robots/fr3/dynamics.yaml')}"
+            dynamics="${xacro.load_yaml('$(arg fr3_dynamics_path)')}"
             accelerometer_config="${xacro.load_yaml('$(find franka_description)/mjcf/robots/fr3/accelerometers.yaml')}"
             hand="$(arg hand)"
@@ -133,5 +138,5 @@
     <default>
         <default class="$(arg arm_id)">
-            <joint armature="0.1" damping="1"/>
+            <joint armature="$(arg fr3_armature)" damping="1"/>
             <position inheritrange="1"/>
             <default class="visual">
